Commit message: updating URDF to include distance sensors

File: robomagellan/models/corobot1.urdf (robot description, URDF)
Before this commit: robot robomagellan, 4 links, 3 joints
Links:
- added link infrared_1; visual box size=0.02 0.01 0.01
- added link ultrasonic_1; visual box size=0.02 0.01 0.01
- added link ultrasonic_2; visual box size=0.02 0.01 0.01
- added link ultrasonic_3; visual box size=0.02 0.01 0.01
- added link ultrasonic_4; visual box size=0.02 0.01 0.01
Joints:
- added joint base_link_to_infrared_1: type fixed, parent base_link, child infrared_1, origin xyz=0.25 0.0 -0.08
- added joint base_link_to_ultrasonic_1: type fixed, parent base_link, child ultrasonic_1, origin xyz=0.20 -0.083 0.125 rpy=0.0 0.0 -0.18
- added joint base_link_to_ultrasonic_2: type fixed, parent base_link, child ultrasonic_2, origin xyz=0.25 -0.042 0.125
- added joint base_link_to_ultrasonic_3: type fixed, parent base_link, child ultrasonic_3, origin xyz=0.25 0.042 0.125
- added joint base_link_to_ultrasonic_4: type fixed, parent base_link, child ultrasonic_4, origin xyz=0.20 0.083 0.125 rpy=0.0 0.0 0.18
