Commit message: use xacro now

File: robomagellan/models/corobot1.urdf.xacro (robot description, xacro)
@@ -1,7 +1,9 @@
 <?xml version="1.0"?>
-<robot name="robomagellan">
+<robot xmlns:xacro="http://www.ros.org/wiki/xacro" name="robomagellan">
+	<xacro:property name="centerToAxle" value="0.2" />
+	<xacro:property name="groundToAxle" value="0.06" />
 	<link name="base_footprint">
 		<!--
-			Attaches the base_link to the ground
+			Attaches the robot to the world frame
 		 -->
 	</link>
@@ -80,5 +82,5 @@
 		<parent link="base_footprint"/>
 		<child link="base_link"/>
-		<origin xyz="0.0 0.0 0.125" />
+		<origin xyz="${-1 * centerToAxle} 0.0 ${groundToAxle}" />
 	</joint>
 	<joint name="base_link_to_camera_lens" type="fixed">

Commit message: corrected the measurements and located the frames

File: robomagellan/models/corobot1.urdf.xacro (robot description, xacro)
@@ -2,26 +2,71 @@
 <robot xmlns:xacro="http://www.ros.org/wiki/xacro" name="robomagellan">
 	<xacro:property name="centerToAxle" value="0.2" />
-	<xacro:property name="groundToAxle" value="0.06" />
-	<link name="base_footprint">
-		<!--
-			Attaches the robot to the world frame
-		 -->
-	</link>
+    <material name="blue">
+        <color rgba="0 0 1 1"/>
+    </material>
+    <material name="red">
+        <color rgba="1 0 0 1"/>
+    </material>
+    <material name="green">
+        <color rgba="0 1 0 1"/>
+    </material>
+    <material name="yellow">
+        <color rgba="0 0.5 0.5 1"/>
+    </material>
+	<link name="base_footprint"/>
+	<joint name="base_footprint_to_base_link" type="fixed">
+		<parent link="base_footprint"/>
+		<child link="base_link"/>
+		<origin xyz="0.093 0.0 0.055" />
+	</joint>
 	<link name="base_link">
-		<!--
-			The base of the robot itself.
-			The GPS and IMU are also linked to this frame
-		 -->
 		<visual>
+			<origin xyz="-0.093 0.0 0.072" rpy="0 0 0" />
 			<geometry>
-				<box size="0.5 0.25 0.25" />
+				<box size="0.295 0.22 0.184" />
 			</geometry>
-			<material name="blue">
-				<color rgba="0 0 1 1"/>
-			</material>
+			<material name="blue"/>
 		</visual>
 	</link>
+	<joint name="base_link_to_left_wheel" type="fixed">
+		<parent link="base_link"/>
+		<child link="left_wheel"/>
+		<origin xyz="0.0 0.135 0.0" />
+	</joint>
+	<link name="left_wheel">
+		<visual>
+			<origin xyz="0.0 0.0 0.0" rpy="1.570 0 0" />
+			<geometry>
+				<cylinder radius="0.055" length="0.053" />
+			</geometry>
+			<material name="red"/>
+		</visual>
+	</link>
+	<joint name="base_link_to_right_wheel" type="fixed">
+		<parent link="base_link"/>
+		<child link="right_wheel"/>
+		<origin xyz="0.0 -0.135 0.0" />
+	</joint>
+	<link name="right_wheel">
+		<visual>
+			<origin xyz="0.0 0.0 0.0" rpy="-1.570 0 0" />
+			<geometry>
+				<cylinder radius="0.055" length="0.053" />
+			</geometry>
+			<material name="red"/>
+		</visual>
+	</link>
+	<joint name="base_link_to_camera_lens" type="fixed">
+		<parent link="base_link"/>
+		<child link="camera_lens"/>
+		<origin xyz="0.035 0.035 0.199" />
+	</joint>
 	<link name="camera_lens">
 	</link>
+	<joint name="camera_lens_to_camera_lens_optical" type="fixed">
+		<parent link="camera_lens"/>
+		<child link="camera_lens_optical"/>
+		<origin xyz="0 0 0" rpy="0.0 1.57 0.0" />
+	</joint>
 	<link name="camera_lens_optical">
 		<visual>
@@ -29,93 +74,71 @@
 				<cylinder radius="0.01" length="0.02" />
 			</geometry>
-			<material name="red">
-				<color rgba="1 0 0 1"/>
-			</material>
+			<material name="red"/>
 		</visual>
 	</link>
-	<link name="ultrasonic_1">
-	    <!-- the left-most ultrasonic rangefinder -->
+    <joint name="base_link_to_infrared_1" type="fixed">
+        <parent link="base_link"/>
+        <child link="infrared_1"/>
+        <origin xyz="0.040 0.0 0.0"/>
+    </joint>
+	<link name="infrared_1">
 		<visual>
 			<geometry>
-				<box size="0.02 0.01 0.01" />
+				<box size="0.01 0.032 0.013" />
 			</geometry>
-			<material name="green">
-				<color rgba="0 1 0 1"/>
-			</material>
+			<material name="yellow"/>
 		</visual>
 	</link>
-	<link name="ultrasonic_2">
+    <joint name="base_link_to_ultrasonic_1" type="fixed">
+        <parent link="base_link"/>
+        <child link="ultrasonic_1"/>
+        <origin xyz="0.060 -0.040 0.145" rpy="0.0 0.0 0.0"/>
+    </joint>
+	<link name="ultrasonic_1">
 		<visual>
 			<geometry>
-				<box size="0.02 0.01 0.01" />
+				<box size="0.015 0.047 0.025" />
 			</geometry>
 			<material name="green"/>
 		</visual>
 	</link>
-	<link name="ultrasonic_3">
+    <joint name="base_link_to_ultrasonic_2" type="fixed">
+        <parent link="base_link"/>
+        <child link="ultrasonic_2"/>
+        <origin xyz="0.060 0.040 0.145" rpy="0.0 0.0 0.0"/>
+    </joint>
+	<link name="ultrasonic_2">
 		<visual>
 			<geometry>
-				<box size="0.02 0.01 0.01" />
+				<box size="0.015 0.047 0.025" />
 			</geometry>
 			<material name="green"/>
 		</visual>
 	</link>
-	<link name="ultrasonic_4">
+    <joint name="base_link_to_ultrasonic_3" type="fixed">
+        <parent link="base_link"/>
+        <child link="ultrasonic_3"/>
+        <origin xyz="0.055 -0.090 0.145" rpy="0.0 0.0 -0.349"/>
+    </joint>
+	<link name="ultrasonic_3">
 		<visual>
 			<geometry>
-				<box size="0.02 0.01 0.01" />
+				<box size="0.015 0.047 0.025" />
 			</geometry>
 			<material name="green"/>
 		</visual>
 	</link>
-	<link name="infrared_1">
-		<visual>
-			<geometry>
-				<box size="0.02 0.01 0.01" />
-			</geometry>
-			<material name="yellow">
-				<color rgba="0 0.5 0.5 1"/>
-			</material>
-		</visual>
-	</link>
-	<joint name="base_footprint_to_base_link" type="fixed">
-		<parent link="base_footprint"/>
-		<child link="base_link"/>
-		<origin xyz="${-1 * centerToAxle} 0.0 ${groundToAxle}" />
-	</joint>
-	<joint name="base_link_to_camera_lens" type="fixed">
-		<parent link="base_link"/>
-		<child link="camera_lens"/>
-		<origin xyz="0.25 0.0 0.125" />
-	</joint>
-	<joint name="camera_lens_to_camera_lens_optical" type="fixed">
-		<parent link="camera_lens"/>
-		<child link="camera_lens_optical"/>
-		<origin xyz="0 0 0" rpy="-1.57 0 -1.57" />
-	</joint>
-    <joint name="base_link_to_infrared_1" type="fixed">
-        <parent link="base_link"/>
-        <child link="infrared_1"/>
-        <origin xyz="0.25 0.0 -0.08"/>
-    </joint>
-    <joint name="base_link_to_ultrasonic_1" type="fixed">
-        <parent link="base_link"/>
-        <child link="ultrasonic_1"/>
-        <origin xyz="0.20 -0.083 0.125" rpy="0.0 0.0 -0.18"/>
-    </joint>
-    <joint name="base_link_to_ultrasonic_2" type="fixed">
-        <parent link="base_link"/>
-        <child link="ultrasonic_2"/>
-        <origin xyz="0.25 -0.042 0.125"/>
-    </joint>
-    <joint name="base_link_to_ultrasonic_3" type="fixed">
-        <parent link="base_link"/>
-        <child link="ultrasonic_3"/>
-        <origin xyz="0.25 0.042 0.125"/>
-    </joint>
     <joint name="base_link_to_ultrasonic_4" type="fixed">
         <parent link="base_link"/>
         <child link="ultrasonic_4"/>
-        <origin xyz="0.20 0.083 0.125" rpy="0.0 0.0 0.18"/>
+        <origin xyz="0.055 0.090 0.145" rpy="0.0 0.0 0.349"/>
     </joint>
+	<link name="ultrasonic_4">
+		<visual>
+			<geometry>
+				<box size="0.015 0.047 0.025" />
+			</geometry>
+			<material name="green"/>
+		</visual>
+	</link>
 </robot>

Commit message: placed the ultrasonic on their frame, corrected other measurements

File: robomagellan/models/corobot1.urdf.xacro (robot description, xacro)
@@ -1,5 +1,7 @@
 <?xml version="1.0"?>
 <robot xmlns:xacro="http://www.ros.org/wiki/xacro" name="robomagellan">
-	<xacro:property name="centerToAxle" value="0.2" />
+	<xacro:property name="mainLength" value="0.295" />
+	<xacro:property name="mainWidth" value="0.220" />
+	<xacro:property name="mainHeight" value="0.184" />
     <material name="blue">
         <color rgba="0 0 1 1"/>
@@ -24,5 +26,5 @@
 			<origin xyz="-0.093 0.0 0.072" rpy="0 0 0" />
 			<geometry>
-				<box size="0.295 0.22 0.184" />
+				<box size="${mainLength} ${mainWidth} ${mainHeight}" />
 			</geometry>
 			<material name="blue"/>
@@ -80,5 +82,5 @@
         <parent link="base_link"/>
         <child link="infrared_1"/>
-        <origin xyz="0.040 0.0 0.0"/>
+        <origin xyz="0.047 0.0 0.005"/>
     </joint>
 	<link name="infrared_1">
@@ -93,5 +95,5 @@
         <parent link="base_link"/>
         <child link="ultrasonic_1"/>
-        <origin xyz="0.060 -0.040 0.145" rpy="0.0 0.0 0.0"/>
+        <origin xyz="0.090 -0.038 0.185" rpy="0.0 0.0 0.0"/>
     </joint>
 	<link name="ultrasonic_1">
@@ -106,5 +108,5 @@
         <parent link="base_link"/>
         <child link="ultrasonic_2"/>
-        <origin xyz="0.060 0.040 0.145" rpy="0.0 0.0 0.0"/>
+        <origin xyz="0.090 0.041 0.185" rpy="0.0 0.0 0.0"/>
     </joint>
 	<link name="ultrasonic_2">
@@ -119,5 +121,5 @@
         <parent link="base_link"/>
         <child link="ultrasonic_3"/>
-        <origin xyz="0.055 -0.090 0.145" rpy="0.0 0.0 -0.349"/>
+        <origin xyz="0.090 -0.100 0.185" rpy="0.0 0.0 -0.052"/>
     </joint>
 	<link name="ultrasonic_3">
@@ -132,5 +134,5 @@
         <parent link="base_link"/>
         <child link="ultrasonic_4"/>
-        <origin xyz="0.055 0.090 0.145" rpy="0.0 0.0 0.349"/>
+        <origin xyz="0.090 0.105 0.185" rpy="0.0 0.0 0.035"/>
     </joint>
 	<link name="ultrasonic_4">
