Commit message: increasing resolution of poor mans laser scanner

File: robomagellan/models/nomad1.urdf.xacro (robot description, xacro)
@@ -92,4 +92,18 @@
 		</visual>
 	</link>
+    <!-- the theoretical center of our ultrasonic array -->
+    <joint name="base_link_to_base_laser_link" type="fixed">
+        <parent link="base_link"/>
+        <child link="base_laser_link"/>
+        <origin xyz="0.090 0.0 0.185" rpy="0.0 0.0 0.0"/>
+    </joint>
+	<link name="base_laser_link">
+		<visual>
+			<geometry>
+				<box size="0.015 0.047 0.025" />
+			</geometry>
+			<material name="green"/>
+		</visual>
+	</link>
     <joint name="base_link_to_ultrasonic_1" type="fixed">
         <parent link="base_link"/>

Commit message: relocated camera frame

File: robomagellan/models/nomad1.urdf.xacro (robot description, xacro)
@@ -62,5 +62,5 @@
 		<parent link="base_link"/>
 		<child link="camera_lens"/>
-		<origin xyz="0.035 0.035 0.199" />
+		<origin xyz="0.100 0.044 0.083" />
 	</joint>
 	<link name="camera_lens">

Commit message: renamed foward infrared frame

File: robomagellan/models/nomad1.urdf.xacro (robot description, xacro)
@@ -84,5 +84,5 @@
         <origin xyz="0.047 0.0 0.005"/>
     </joint>
-	<link name="infrared_1">
+	<link name="infrared_forward">
 		<visual>
 			<geometry>

Commit message: renamed infrared frame

File: robomagellan/models/nomad1.urdf.xacro (robot description, xacro)
@@ -1,7 +1,7 @@
 <?xml version="1.0"?>
 <robot xmlns:xacro="http://www.ros.org/wiki/xacro" name="robomagellan">
-	<xacro:property name="mainLength" value="0.295" />
-	<xacro:property name="mainWidth" value="0.220" />
-	<xacro:property name="mainHeight" value="0.184" />
+    <xacro:property name="mainLength" value="0.295" />
+    <xacro:property name="mainWidth" value="0.220" />
+    <xacro:property name="mainHeight" value="0.184" />
     <material name="blue">
         <color rgba="0 0 1 1"/>
@@ -16,80 +16,80 @@
         <color rgba="0 0.5 0.5 1"/>
     </material>
-	<link name="base_footprint"/>
-	<joint name="base_footprint_to_base_link" type="fixed">
-		<parent link="base_footprint"/>
-		<child link="base_link"/>
-		<origin xyz="0.093 0.0 0.055" />
-	</joint>
-	<link name="base_link">
-		<visual>
-			<origin xyz="-0.093 0.0 0.072" rpy="0 0 0" />
-			<geometry>
-				<box size="${mainLength} ${mainWidth} ${mainHeight}" />
-			</geometry>
-			<material name="blue"/>
-		</visual>
-	</link>
-	<joint name="base_link_to_left_wheel" type="fixed">
-		<parent link="base_link"/>
-		<child link="left_wheel"/>
-		<origin xyz="0.0 0.135 0.0" />
-	</joint>
-	<link name="left_wheel">
-		<visual>
-			<origin xyz="0.0 0.0 0.0" rpy="1.570 0 0" />
-			<geometry>
-				<cylinder radius="0.055" length="0.053" />
-			</geometry>
-			<material name="red"/>
-		</visual>
-	</link>
-	<joint name="base_link_to_right_wheel" type="fixed">
-		<parent link="base_link"/>
-		<child link="right_wheel"/>
-		<origin xyz="0.0 -0.135 0.0" />
-	</joint>
-	<link name="right_wheel">
-		<visual>
-			<origin xyz="0.0 0.0 0.0" rpy="-1.570 0 0" />
-			<geometry>
-				<cylinder radius="0.055" length="0.053" />
-			</geometry>
-			<material name="red"/>
-		</visual>
-	</link>
-	<joint name="base_link_to_camera_lens" type="fixed">
-		<parent link="base_link"/>
-		<child link="camera_lens"/>
-		<origin xyz="0.100 0.044 0.083" />
-	</joint>
-	<link name="camera_lens">
-	</link>
-	<joint name="camera_lens_to_camera_lens_optical" type="fixed">
-		<parent link="camera_lens"/>
-		<child link="camera_lens_optical"/>
-		<origin xyz="0 0 0" rpy="0.0 1.57 0.0" />
-	</joint>
-	<link name="camera_lens_optical">
-		<visual>
-			<geometry>
-				<cylinder radius="0.01" length="0.02" />
-			</geometry>
-			<material name="red"/>
-		</visual>
-	</link>
-    <joint name="base_link_to_infrared_1" type="fixed">
+    <link name="base_footprint"/>
+    <joint name="base_footprint_to_base_link" type="fixed">
+        <parent link="base_footprint"/>
+        <child link="base_link"/>
+        <origin xyz="0.093 0.0 0.055" />
+    </joint>
+    <link name="base_link">
+        <visual>
+            <origin xyz="-0.093 0.0 0.072" rpy="0 0 0" />
+            <geometry>
+                <box size="${mainLength} ${mainWidth} ${mainHeight}" />
+            </geometry>
+            <material name="blue"/>
+        </visual>
+    </link>
+    <joint name="base_link_to_left_wheel" type="fixed">
         <parent link="base_link"/>
-        <child link="infrared_1"/>
+        <child link="left_wheel"/>
+        <origin xyz="0.0 0.135 0.0" />
+    </joint>
+    <link name="left_wheel">
+        <visual>
+            <origin xyz="0.0 0.0 0.0" rpy="1.570 0 0" />
+            <geometry>
+                <cylinder radius="0.055" length="0.053" />
+            </geometry>
+            <material name="red"/>
+        </visual>
+    </link>
+    <joint name="base_link_to_right_wheel" type="fixed">
+        <parent link="base_link"/>
+        <child link="right_wheel"/>
+        <origin xyz="0.0 -0.135 0.0" />
+    </joint>
+    <link name="right_wheel">
+        <visual>
+            <origin xyz="0.0 0.0 0.0" rpy="-1.570 0 0" />
+            <geometry>
+                <cylinder radius="0.055" length="0.053" />
+            </geometry>
+            <material name="red"/>
+        </visual>
+    </link>
+    <joint name="base_link_to_camera_lens" type="fixed">
+        <parent link="base_link"/>
+        <child link="camera_lens"/>
+        <origin xyz="0.100 0.044 0.083" />
+    </joint>
+    <link name="camera_lens">
+    </link>
+    <joint name="camera_lens_to_camera_lens_optical" type="fixed">
+        <parent link="camera_lens"/>
+        <child link="camera_lens_optical"/>
+        <origin xyz="0 0 0" rpy="0.0 1.57 0.0" />
+    </joint>
+    <link name="camera_lens_optical">
+        <visual>
+            <geometry>
+                <cylinder radius="0.01" length="0.02" />
+            </geometry>
+            <material name="red"/>
+        </visual>
+    </link>
+    <joint name="base_link_to_infrared_forward" type="fixed">
+        <parent link="base_link"/>
+        <child link="infrared_forward"/>
         <origin xyz="0.047 0.0 0.005"/>
     </joint>
-	<link name="infrared_forward">
-		<visual>
-			<geometry>
-				<box size="0.01 0.032 0.013" />
-			</geometry>
-			<material name="yellow"/>
-		</visual>
-	</link>
+    <link name="infrared_forward">
+        <visual>
+            <geometry>
+                <box size="0.01 0.032 0.013" />
+            </geometry>
+            <material name="yellow"/>
+        </visual>
+    </link>
     <!-- the theoretical center of our ultrasonic array -->
     <joint name="base_link_to_base_laser_link" type="fixed">
@@ -98,12 +98,12 @@
         <origin xyz="0.090 0.0 0.185" rpy="0.0 0.0 0.0"/>
     </joint>
-	<link name="base_laser_link">
-		<visual>
-			<geometry>
-				<box size="0.015 0.047 0.025" />
-			</geometry>
-			<material name="green"/>
-		</visual>
-	</link>
+    <link name="base_laser_link">
+        <visual>
+            <geometry>
+                <box size="0.015 0.047 0.025" />
+            </geometry>
+            <material name="green"/>
+        </visual>
+    </link>
     <joint name="base_link_to_ultrasonic_1" type="fixed">
         <parent link="base_link"/>
@@ -111,12 +111,12 @@
         <origin xyz="0.090 -0.038 0.185" rpy="0.0 0.0 0.0"/>
     </joint>
-	<link name="ultrasonic_1">
-		<visual>
-			<geometry>
-				<box size="0.015 0.047 0.025" />
-			</geometry>
-			<material name="green"/>
-		</visual>
-	</link>
+    <link name="ultrasonic_1">
+        <visual>
+            <geometry>
+                <box size="0.015 0.047 0.025" />
+            </geometry>
+            <material name="green"/>
+        </visual>
+    </link>
     <joint name="base_link_to_ultrasonic_2" type="fixed">
         <parent link="base_link"/>
@@ -124,12 +124,12 @@
         <origin xyz="0.090 0.041 0.185" rpy="0.0 0.0 0.0"/>
     </joint>
-	<link name="ultrasonic_2">
-		<visual>
-			<geometry>
-				<box size="0.015 0.047 0.025" />
-			</geometry>
-			<material name="green"/>
-		</visual>
-	</link>
+    <link name="ultrasonic_2">
+        <visual>
+            <geometry>
+                <box size="0.015 0.047 0.025" />
+            </geometry>
+            <material name="green"/>
+        </visual>
+    </link>
     <joint name="base_link_to_ultrasonic_3" type="fixed">
         <parent link="base_link"/>
@@ -137,12 +137,12 @@
         <origin xyz="0.090 -0.100 0.185" rpy="0.0 0.0 -0.052"/>
     </joint>
-	<link name="ultrasonic_3">
-		<visual>
-			<geometry>
-				<box size="0.015 0.047 0.025" />
-			</geometry>
-			<material name="green"/>
-		</visual>
-	</link>
+    <link name="ultrasonic_3">
+        <visual>
+            <geometry>
+                <box size="0.015 0.047 0.025" />
+            </geometry>
+            <material name="green"/>
+        </visual>
+    </link>
     <joint name="base_link_to_ultrasonic_4" type="fixed">
         <parent link="base_link"/>
@@ -150,11 +150,11 @@
         <origin xyz="0.090 0.105 0.185" rpy="0.0 0.0 0.035"/>
     </joint>
-	<link name="ultrasonic_4">
-		<visual>
-			<geometry>
-				<box size="0.015 0.047 0.025" />
-			</geometry>
-			<material name="green"/>
-		</visual>
-	</link>
+    <link name="ultrasonic_4">
+        <visual>
+            <geometry>
+                <box size="0.015 0.047 0.025" />
+            </geometry>
+            <material name="green"/>
+        </visual>
+    </link>
 </robot>

Commit message: fore and aft infrared sensors

File: robomagellan/models/nomad1.urdf.xacro (robot description, xacro)
@@ -92,4 +92,17 @@
         </visual>
     </link>
+    <joint name="base_link_to_infrared_aft" type="fixed">
+        <parent link="base_link"/>
+        <child link="infrared_aft"/>
+        <origin xyz="-0.23 0.0 0.034" rpy="0.0 0.0 3.1415"/>
+    </joint>
+    <link name="infrared_aft">
+        <visual>
+            <geometry>
+                <box size="0.01 0.032 0.013" />
+            </geometry>
+            <material name="yellow"/>
+        </visual>
+    </link>
     <!-- the theoretical center of our ultrasonic array -->
     <joint name="base_link_to_base_laser_link" type="fixed">

Commit message: repositioned the camera

File: robomagellan/models/nomad1.urdf.xacro (robot description, xacro)
@@ -62,5 +62,5 @@
         <parent link="base_link"/>
         <child link="camera_lens"/>
-        <origin xyz="0.100 0.044 0.083" />
+        <origin xyz="0.065 0.000 0.203" />
     </joint>
     <link name="camera_lens">

Commit message: adding imu frame

File: robomagellan/models/nomad1.urdf.xacro (robot description, xacro)
@@ -57,4 +57,18 @@
             </geometry>
             <material name="red"/>
+        </visual>
+    </link>
+    <joint name="base_link_to_imu" type="fixed">
+        <parent link="base_link"/>
+        <child link="imu"/>
+        <origin xyz="-0.18 -0.065 1.095" />
+    </joint>
+    <link name="imu">
+        <visual>
+            <origin xyz="0.0 0.0 0.0" rpy="0 0 0" />
+            <geometry>
+                <cylinder radius="0.055" length="0.053" />
+            </geometry>
+            <material name="blue"/>
         </visual>
     </link>

Commit message: update urdf after moving IMU

File: robomagellan/models/nomad1.urdf.xacro (robot description, xacro)
@@ -62,5 +62,5 @@
         <parent link="base_link"/>
         <child link="imu"/>
-        <origin xyz="-0.18 -0.065 1.095" />
+        <origin xyz="-0.098 0.110 1.125" />
     </joint>
     <link name="imu">

Commit message: parameter for imuHeight and parameterized ultrasonics and imu

File: robomagellan/models/nomad1.urdf.xacro (robot description, xacro)
@@ -4,4 +4,7 @@
     <xacro:property name="mainWidth" value="0.220" />
     <xacro:property name="mainHeight" value="0.184" />
+    <xacro:property name="axleHeight" value="0.049" />
+    <xacro:property name="imuHeight" value="1.165" />
+    <xacro:property name="ultrasonicHeight" value="0.230" />
     <material name="blue">
         <color rgba="0 0 1 1"/>
@@ -20,5 +23,5 @@
         <parent link="base_footprint"/>
         <child link="base_link"/>
-        <origin xyz="0.093 0.0 0.055" />
+        <origin xyz="0.093 0.0 ${axleHeight}" />
     </joint>
     <link name="base_link">
@@ -62,5 +65,5 @@
         <parent link="base_link"/>
         <child link="imu"/>
-        <origin xyz="-0.098 0.110 1.125" />
+        <origin xyz="-0.098 0.110 ${imuHeight-axleHeight}" />
     </joint>
     <link name="imu">
@@ -123,5 +126,5 @@
         <parent link="base_link"/>
         <child link="base_laser_link"/>
-        <origin xyz="0.090 0.0 0.185" rpy="0.0 0.0 0.0"/>
+        <origin xyz="0.090 0.0 ${ultrasonicHeight-axleHeight}" rpy="0.0 0.0 0.0"/>
     </joint>
     <link name="base_laser_link">
@@ -136,5 +139,5 @@
         <parent link="base_link"/>
         <child link="ultrasonic_1"/>
-        <origin xyz="0.090 -0.038 0.185" rpy="0.0 0.0 0.0"/>
+        <origin xyz="0.090 -0.038 ${ultrasonicHeight-axleHeight}" rpy="0.0 0.0 0.0"/>
     </joint>
     <link name="ultrasonic_1">
@@ -149,5 +152,5 @@
         <parent link="base_link"/>
         <child link="ultrasonic_2"/>
-        <origin xyz="0.090 0.041 0.185" rpy="0.0 0.0 0.0"/>
+        <origin xyz="0.090 0.041 ${ultrasonicHeight-axleHeight}" rpy="0.0 0.0 0.0"/>
     </joint>
     <link name="ultrasonic_2">
@@ -162,5 +165,5 @@
         <parent link="base_link"/>
         <child link="ultrasonic_3"/>
-        <origin xyz="0.090 -0.100 0.185" rpy="0.0 0.0 -0.052"/>
+        <origin xyz="0.090 -0.100 ${ultrasonicHeight-axleHeight}" rpy="0.0 0.0 -0.052"/>
     </joint>
     <link name="ultrasonic_3">
@@ -175,5 +178,5 @@
         <parent link="base_link"/>
         <child link="ultrasonic_4"/>
-        <origin xyz="0.090 0.105 0.185" rpy="0.0 0.0 0.035"/>
+        <origin xyz="0.090 0.105 ${ultrasonicHeight-axleHeight}" rpy="0.0 0.0 0.035"/>
     </joint>
     <link name="ultrasonic_4">

Commit message: added timestamps to motors_c and lowered IMU

File: robomagellan/models/nomad1.urdf.xacro (robot description, xacro)
@@ -5,5 +5,5 @@
     <xacro:property name="mainHeight" value="0.184" />
     <xacro:property name="axleHeight" value="0.049" />
-    <xacro:property name="imuHeight" value="1.165" />
+    <xacro:property name="imuHeight" value="0.743" />
     <xacro:property name="ultrasonicHeight" value="0.230" />
     <material name="blue">

Commit message: replaced ultrasonic with laser

File: robomagellan/models/nomad1.urdf.xacro (robot description, xacro)
@@ -6,5 +6,5 @@
     <xacro:property name="axleHeight" value="0.049" />
     <xacro:property name="imuHeight" value="0.743" />
-    <xacro:property name="ultrasonicHeight" value="0.230" />
+    <xacro:property name="laserHeight" value="0.270" />
     <material name="blue">
         <color rgba="0 0 1 1"/>
@@ -122,66 +122,14 @@
         </visual>
     </link>
-    <!-- the theoretical center of our ultrasonic array -->
-    <joint name="base_link_to_base_laser_link" type="fixed">
+    <joint name="base_link_to_laser" type="fixed">
         <parent link="base_link"/>
         <child link="base_laser_link"/>
-        <origin xyz="0.090 0.0 ${ultrasonicHeight-axleHeight}" rpy="0.0 0.0 0.0"/>
+        <origin xyz="0.010 0.004 ${laserHeight-axleHeight}"
+                rpy="0.0 0.0 -0.02"/>
     </joint>
-    <link name="base_laser_link">
+    <link name="laser">
         <visual>
             <geometry>
-                <box size="0.015 0.047 0.025" />
-            </geometry>
-            <material name="green"/>
-        </visual>
-    </link>
-    <joint name="base_link_to_ultrasonic_1" type="fixed">
-        <parent link="base_link"/>
-        <child link="ultrasonic_1"/>
-        <origin xyz="0.090 -0.038 ${ultrasonicHeight-axleHeight}" rpy="0.0 0.0 0.0"/>
-    </joint>
-    <link name="ultrasonic_1">
-        <visual>
-            <geometry>
-                <box size="0.015 0.047 0.025" />
-            </geometry>
-            <material name="green"/>
-        </visual>
-    </link>
-    <joint name="base_link_to_ultrasonic_2" type="fixed">
-        <parent link="base_link"/>
-        <child link="ultrasonic_2"/>
-        <origin xyz="0.090 0.041 ${ultrasonicHeight-axleHeight}" rpy="0.0 0.0 0.0"/>
-    </joint>
-    <link name="ultrasonic_2">
-        <visual>
-            <geometry>
-                <box size="0.015 0.047 0.025" />
-            </geometry>
-            <material name="green"/>
-        </visual>
-    </link>
-    <joint name="base_link_to_ultrasonic_3" type="fixed">
-        <parent link="base_link"/>
-        <child link="ultrasonic_3"/>
-        <origin xyz="0.090 -0.100 ${ultrasonicHeight-axleHeight}" rpy="0.0 0.0 -0.052"/>
-    </joint>
-    <link name="ultrasonic_3">
-        <visual>
-            <geometry>
-                <box size="0.015 0.047 0.025" />
-            </geometry>
-            <material name="green"/>
-        </visual>
-    </link>
-    <joint name="base_link_to_ultrasonic_4" type="fixed">
-        <parent link="base_link"/>
-        <child link="ultrasonic_4"/>
-        <origin xyz="0.090 0.105 ${ultrasonicHeight-axleHeight}" rpy="0.0 0.0 0.035"/>
-    </joint>
-    <link name="ultrasonic_4">
-        <visual>
-            <geometry>
-                <box size="0.015 0.047 0.025" />
+                <box size="0.060 0.060 0.085" />
             </geometry>
             <material name="green"/>

Commit message: replaced ultrasonic array with hokuyo

File: robomagellan/models/nomad1.urdf.xacro (robot description, xacro)
@@ -124,5 +124,5 @@
     <joint name="base_link_to_laser" type="fixed">
         <parent link="base_link"/>
-        <child link="base_laser_link"/>
+        <child link="laser"/>
         <origin xyz="0.010 0.004 ${laserHeight-axleHeight}"
                 rpy="0.0 0.0 -0.02"/>
